Commit message: fix gp mpc

File: src/ros_gp_mpc/config/hummingbird.xacro (robot description, xacro)
@@ -19,25 +19,28 @@
   <!-- Properties (Taken from Novel Dynamic Inversion Architecture Design
 for Quadrocopter Control by Jian Wang et al.) -->
+  <!-- Properties -->
   <xacro:property name="namespace" value="$(arg namespace)" />
   <xacro:property name="rotor_velocity_slowdown_sim" value="10" />
   <xacro:property name="use_mesh_file" value="true" />
-  <xacro:property name="mesh_file" value="package://rotors_description/meshes/hummingbird.dae" />
-  <xacro:property name="mass" value="0.68" /> <!-- [kg] -->
+  <xacro:property name="mesh_file" value="package://rotors_description/meshes/firefly.dae" />
+  <xacro:property name="mass" value="0.09" /> <!-- [kg] -->
   <xacro:property name="body_width" value="0.1" /> <!-- [m] -->
-  <xacro:property name="body_height" value="0.12" /> <!-- [m] -->
-  <xacro:property name="mass_rotor" value="0.009" /> <!-- [kg] -->
-  <xacro:property name="arm_length" value="0.17" /> <!-- [m] -->
-  <xacro:property name="rotor_offset_top" value="0.01" /> <!-- 0.01 [m] -->
+  <xacro:property name="body_height" value="0.16" /> <!-- [m] -->
+  <xacro:property name="mass_rotor" value="0.005" /> <!-- [kg] -->
+  <xacro:property name="arm_length" value="0.04" /> <!-- [m] -->
+  <xacro:property name="rotor_offset_top" value="0.037" /> <!-- [m] -->
   <xacro:property name="radius_rotor" value="0.1" /> <!-- [m] -->
   <xacro:property name="motor_constant" value="8.54858e-06" /> <!-- [kg m/s^2] -->
-  <xacro:property name="moment_constant" value="0.05" /> <!-- [m] 0.016-->
+  <xacro:property name="moment_constant" value="0.016" /> <!-- [m] -->
   <xacro:property name="time_constant_up" value="0.0125" /> <!-- [s] -->
   <xacro:property name="time_constant_down" value="0.025" /> <!-- [s] -->
   <xacro:property name="max_rot_velocity" value="838" /> <!-- [rad/s] -->
-  <xacro:property name="rotor_drag_coefficient" value="8.06428e-05" /> <!-- 8.06428e-05 -->
+  <xacro:property name="sin30" value="0.5" />
+  <xacro:property name="cos30" value="0.866025403784" />
+  <xacro:property name="rotor_drag_coefficient" value="8.06428e-05" />
   <xacro:property name="rolling_moment_coefficient" value="0.000001" />
   <!-- Property Blocks -->
   <xacro:property name="body_inertia">
-    <inertia ixx="0.007" ixy="0.0" ixz="0.0" iyy="0.007" iyz="0.0" izz="0.012" /> <!-- [kg m^2] [kg m^2] [kg m^2] [kg m^2] [kg m^2] [kg m^2] -->
+    <inertia ixx="0.00059" ixy="0.0" ixz="0.0" iyy="0.00059" iyz="0.0" izz="0.00059" /> <!-- [kg m^2] [kg m^2] [kg m^2] [kg m^2] [kg m^2] [kg m^2] -->
   </xacro:property>
   <!-- inertia of a single rotor, assuming it is a cuboid. Height=3mm, width=15mm -->

File: src/rotors_simulator/rotors_description/urdf/firefly.xacro (robot description, xacro)
@@ -22,9 +22,9 @@
   <xacro:property name="use_mesh_file" value="true" />
   <xacro:property name="mesh_file" value="package://rotors_description/meshes/firefly.dae" />
-  <xacro:property name="mass" value="1.5" /> <!-- [kg] -->
+  <xacro:property name="mass" value="0.09" /> <!-- [kg] -->
   <xacro:property name="body_width" value="0.1" /> <!-- [m] -->
   <xacro:property name="body_height" value="0.16" /> <!-- [m] -->
   <xacro:property name="mass_rotor" value="0.005" /> <!-- [kg] -->
-  <xacro:property name="arm_length" value="0.215" /> <!-- [m] -->
+  <xacro:property name="arm_length" value="0.04" /> <!-- [m] -->
   <xacro:property name="rotor_offset_top" value="0.037" /> <!-- [m] -->
   <xacro:property name="radius_rotor" value="0.1" /> <!-- [m] -->
@@ -40,5 +40,5 @@
   <!-- Property Blocks -->
   <xacro:property name="body_inertia">
-    <inertia ixx="0.0347563" ixy="0.0" ixz="0.0" iyy="0.0458929" iyz="0.0" izz="0.0977" /> <!-- [kg m^2] [kg m^2] [kg m^2] [kg m^2] [kg m^2] [kg m^2] -->
+    <inertia ixx="0.00059" ixy="0.0" ixz="0.0" iyy="0.00059" iyz="0.0" izz="0.00059" /> <!-- [kg m^2] [kg m^2] [kg m^2] [kg m^2] [kg m^2] [kg m^2] -->
   </xacro:property>
   <!-- inertia of a single rotor, assuming it is a cuboid. Height=3mm, width=15mm -->

Commit message: new

File: src/ros_gp_mpc/config/hummingbird.xacro (robot description, xacro)
@@ -19,28 +19,25 @@
   <!-- Properties (Taken from Novel Dynamic Inversion Architecture Design
 for Quadrocopter Control by Jian Wang et al.) -->
-  <!-- Properties -->
   <xacro:property name="namespace" value="$(arg namespace)" />
   <xacro:property name="rotor_velocity_slowdown_sim" value="10" />
   <xacro:property name="use_mesh_file" value="true" />
-  <xacro:property name="mesh_file" value="package://rotors_description/meshes/firefly.dae" />
-  <xacro:property name="mass" value="0.09" /> <!-- [kg] -->
+  <xacro:property name="mesh_file" value="package://rotors_description/meshes/hummingbird.dae" />
+  <xacro:property name="mass" value="0.68" /> <!-- [kg] -->
   <xacro:property name="body_width" value="0.1" /> <!-- [m] -->
-  <xacro:property name="body_height" value="0.16" /> <!-- [m] -->
-  <xacro:property name="mass_rotor" value="0.005" /> <!-- [kg] -->
-  <xacro:property name="arm_length" value="0.04" /> <!-- [m] -->
-  <xacro:property name="rotor_offset_top" value="0.037" /> <!-- [m] -->
+  <xacro:property name="body_height" value="0.12" /> <!-- [m] -->
+  <xacro:property name="mass_rotor" value="0.009" /> <!-- [kg] -->
+  <xacro:property name="arm_length" value="0.17" /> <!-- [m] -->
+  <xacro:property name="rotor_offset_top" value="0.01" /> <!-- 0.01 [m] -->
   <xacro:property name="radius_rotor" value="0.1" /> <!-- [m] -->
   <xacro:property name="motor_constant" value="8.54858e-06" /> <!-- [kg m/s^2] -->
-  <xacro:property name="moment_constant" value="0.016" /> <!-- [m] -->
+  <xacro:property name="moment_constant" value="0.05" /> <!-- [m] 0.016-->
   <xacro:property name="time_constant_up" value="0.0125" /> <!-- [s] -->
   <xacro:property name="time_constant_down" value="0.025" /> <!-- [s] -->
   <xacro:property name="max_rot_velocity" value="838" /> <!-- [rad/s] -->
-  <xacro:property name="sin30" value="0.5" />
-  <xacro:property name="cos30" value="0.866025403784" />
-  <xacro:property name="rotor_drag_coefficient" value="8.06428e-05" />
+  <xacro:property name="rotor_drag_coefficient" value="8.06428e-05" /> <!-- 8.06428e-05 -->
   <xacro:property name="rolling_moment_coefficient" value="0.000001" />
   <!-- Property Blocks -->
   <xacro:property name="body_inertia">
-    <inertia ixx="0.00059" ixy="0.0" ixz="0.0" iyy="0.00059" iyz="0.0" izz="0.00059" /> <!-- [kg m^2] [kg m^2] [kg m^2] [kg m^2] [kg m^2] [kg m^2] -->
+    <inertia ixx="0.007" ixy="0.0" ixz="0.0" iyy="0.007" iyz="0.0" izz="0.012" /> <!-- [kg m^2] [kg m^2] [kg m^2] [kg m^2] [kg m^2] [kg m^2] -->
   </xacro:property>
   <!-- inertia of a single rotor, assuming it is a cuboid. Height=3mm, width=15mm -->

File: src/rotors_simulator/rotors_description/urdf/firefly.xacro (robot description, xacro)
@@ -22,9 +22,9 @@
   <xacro:property name="use_mesh_file" value="true" />
   <xacro:property name="mesh_file" value="package://rotors_description/meshes/firefly.dae" />
-  <xacro:property name="mass" value="0.09" /> <!-- [kg] -->
+  <xacro:property name="mass" value="1.5" /> <!-- [kg] -->
   <xacro:property name="body_width" value="0.1" /> <!-- [m] -->
   <xacro:property name="body_height" value="0.16" /> <!-- [m] -->
   <xacro:property name="mass_rotor" value="0.005" /> <!-- [kg] -->
-  <xacro:property name="arm_length" value="0.04" /> <!-- [m] -->
+  <xacro:property name="arm_length" value="0.215" /> <!-- [m] -->
   <xacro:property name="rotor_offset_top" value="0.037" /> <!-- [m] -->
   <xacro:property name="radius_rotor" value="0.1" /> <!-- [m] -->
@@ -40,5 +40,5 @@
   <!-- Property Blocks -->
   <xacro:property name="body_inertia">
-    <inertia ixx="0.00059" ixy="0.0" ixz="0.0" iyy="0.00059" iyz="0.0" izz="0.00059" /> <!-- [kg m^2] [kg m^2] [kg m^2] [kg m^2] [kg m^2] [kg m^2] -->
+    <inertia ixx="0.0347563" ixy="0.0" ixz="0.0" iyy="0.0458929" iyz="0.0" izz="0.0977" /> <!-- [kg m^2] [kg m^2] [kg m^2] [kg m^2] [kg m^2] [kg m^2] -->
   </xacro:property>
   <!-- inertia of a single rotor, assuming it is a cuboid. Height=3mm, width=15mm -->
